File: Macropad/macropad.kicad_sch (KiCad schematic)
At the start: 83 parts, among them J1 USB_B_Micro, J2 Conn_01x02, SW1 SW_Push, SW10 SW_Push, SW11 SW_Push, SW12 SW_Push, SW13 SW_Push, SW14 SW_Push, SW15 SW_Push, SW16 SW_Push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

Commit message: macropad: Finish routing - CommsBus - Neopixels
Parts:
- removed J1: USB_B_Micro, RP2040_minimal:USB_Micro-B_Amphenol_10103594-0001LF_Horizontal_modified, symbol Connector:USB_B_Micro
- removed R2: DNF, Resistor_SMD:R_0402_1005Metric, symbol Device:R
- added D34, D35: C8678, Diode_SMD:D_SMA_Handsoldering, symbol Device:D
- added J1: USB_C_Receptacle_USB2.0_14P, Connector_USB:USB_C_Receptacle_G-Switch_GT-USB-7010ASV, symbol Connector:USB_C_Receptacle_USB2.0_14P
- added Q1: A03401A, Package_TO_SOT_SMD:TO-252-2, symbol Transistor_FET:QM6015D
- added R7, R8: 5.1k, Resistor_SMD:R_0805_2012Metric, symbol Device:R_Small
- added R9: 10k, Resistor_SMD:R_0805_2012Metric, symbol Device:R
- C18: footprint Capacitor_SMD:C_0402_1005Metric -> Capacitor_SMD:C_0805_2012Metric
- J2: footprint Connector_PinHeader_2.54mm:PinHeader_1x02_P2.54mm_Vertical -> Connector_PinHeader_2.54mm:PinHeader_1x02_P2.54mm_Horizontal
- R6: footprint Resistor_SMD:R_0402_1005Metric -> Resistor_SMD:R_0805_2012Metric
- U2: footprint Package_SO:SOIC-8_5.23x5.23mm_P1.27mm -> Macropad:SOIC-8_5.23x5.23mm_P1.27mm
Connections:
- net GND: now also J1.A1 (GND), J1.A12 (GND), J1.B1 (GND), J1.B12 (GND), J1.S1 (SHIELD), R7.2, R8.2, R9.2
- net USB_D+: now also J1.A6 (D+), J1.B6 (D+)
- net USB_D-: now also J1.A7 (D-), J1.B7 (D-)
- net VBUS renamed +5V
- net +5V: now also D34.1 (K), Q1.3 (S)
- new net: J1.B5 (CC2), R8.1
- new net: J1.A5 (CC1), R7.1
- new net: D35.1 (K), Q1.2 (D)
- new net EXT5V: D35.2 (A)
- new net USB5V: D34.2 (A), J1.A4 (VBUS), J1.A9 (VBUS), J1.B4 (VBUS), J1.B9 (VBUS), Q1.1 (G), R9.1
- no-connect marks 1 -> 0
Other:
- moved on the sheet: C1, C4, U1
